File: boards/leddriver/leddriver.kicad_pcb (KiCad board)
At the start: 2 copper layers, 37.5 x 49.5 mm, 24 parts, among them K1 CONN_3, K2 CONN_3, P1 CONN_2, P2 CONN_2, P3 CONN_4, Q1 MOS_N, Q2 MOS_N, Q3 MOS_N, U1 LM1117, U2 WS2801

Commit message: Finalized Silkscreen Generated gerbers for production
Parts:
- added G***: logo_hacker_silkbot_20_00mm, logo_hacker_silkbot_20_00mm, B.Cu at (167.0, 134.0)
Other:
- outline, holes or cut-outs redrawn
- board text added: "+"
- board text added: "+12V"
- board text added: "-"
- board text added: "B"
- board text added: "CLKI"
- board text added: "CLKO"
- board text added: "DI"
- board text added: "DO"
- board text added: "G"
- board text added: "GND"
- board text added: "R"
- board text added: "V.0.1"
- board text added: "WS2801 Led Driver"
- board text added: "by Sebastian Schumb 2015"
